File: controller/controller_v0_3.sch (KiCad schematic (older format))
At the start: 30 parts, among them J1 QRSwitch, J2 Screen, J3 Irrigation, J4 EnvSensor, J5 Power, J6 PumpRelay, J7 Condutivity, Q1 Q_NPN_BCE, U1 WeMos_D1_mini, U2 NodeMCU_ESP12E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

Commit message: Production version. First iteration for correction
Parts:
- D3: footprint Diode_THT:D_DO-41_SOD81_P7.62mm_Horizontal -> Diode_THT:D_DO-15_P10.16mm_Horizontal
- Q1: value Q_NPN_BCE -> MPS2222; symbol Device:Q_NPN_BCE -> Device:Q_NPN_EBC
Connections:
- net +5V: no longer D3.1 (K), RLY1.2
- net GND: now also Q1.1 (E); no longer Q1.3 (E)
- net POWER_Vin: now also D3.1 (K), RLY1.2
- net at R6.1, R7.2: now also Q1.2 (B); no longer Q1.1 (B)
- net at D3.2 (A), RLY1.5: now also Q1.3 (C); no longer Q1.2 (C)
Changed lines of the file:
@@
 Title "Hidroponic Controller"
 Date "2021-06-10"
-Rev "v0.2"
+Rev "v0.3"
 Comp "by Luis Pereira"
 Comment1 ""
@@
 Wire Wire Line
 	4600 6050 5000 6050
-$Comp
-L Device:Q_NPN_BCE Q1
-U 1 1 60D0EFE3
-P 3750 6550
-F 0 "Q1" H 3941 6596 50  0000 L CNN
-F 1 "Q_NPN_BCE" H 3941 6505 50  0000 L CNN
-F 2 "Package_TO_SOT_THT:TO-92" H 3950 6650 50  0001 C CNN
-F 3 "~" H 3750 6550 50  0001 C CNN
-	1    3750 6550
-	1    0    0    -1
-$EndComp
 Wire Wire Line
 	3850 6100 3850 6300
@@
 	3850 6800 3900 6800
 Text Label 3850 5600 2    50   ~ 0
-+5V
+POWER_Vin
 Wire Wire Line
 	3850 5800 3850 5700
@@
 F 0 "D3" V 3504 6030 50  0000 L CNN
 F 1 "D" V 3595 6030 50  0000 L CNN
-F 2 "Diode_THT:D_DO-41_SOD81_P7.62mm_Horizontal" H 3550 5950 50  0001 C CNN
+F 2 "Diode_THT:D_DO-15_P10.16mm_Horizontal" H 3550 5950 50  0001 C CNN
 F 3 "~" H 3550 5950 50  0001 C CNN
 	1    3550 5950
@@
 	1    0    0    -1
 $EndComp
+$Comp
+L Device:Q_NPN_EBC Q1
+U 1 1 60D0EFE3
+P 3750 6550
+F 0 "Q1" H 3941 6596 50  0000 L CNN
+F 1 "MPS2222" H 3941 6505 50  0000 L CNN
+F 2 "Package_TO_SOT_THT:TO-92" H 3950 6650 50  0001 C CNN
+F 3 "~" H 3750 6550 50  0001 C CNN
+	1    3750 6550
+	1    0    0    -1
+$EndComp
