File: controller/controller_v0_3.kicad_pcb (KiCad board)
At the start: 2 copper layers, 99.5 x 48.5 mm, 30 parts, among them J1 QRSwitch, J2 Screen, J3 Irrigation, J4 EnvSensor, J5 Power, J6 PumpRelay, J7 Condutivity, Q1 MPS2222, U1 WeMos_D1_mini, U2 NodeMCU_ESP12E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

Commit message: Added version 0.3 with hardware corrections
Other:
- net class Default removed
- net class HV removed
- net class Power removed
